Commit message: Port segmentation_node + Docker dev env + fix upstream refs
PHASE 0 ALGORITHM PORT
  - stem_grasp/segmentation_node.py: full port of the 1096-line ROS 1 node.
    Preserves every parameter, every topic, and the full inference pipeline:
    YOLO-seg, Grounded-SAM (with context prompts + union/best caption modes
    + target caption + 3D backprojection), HSV green fallback, Frangi
    vesselness fusion, depth pre/post filter, mask dilation, instance
    selection (highest_conf / closest_to_base), TF-based closest-mask
    decision, joint_states stationary gate, debug overlay image.
    Mechanical ROS 1->2 swaps only; numpy / cv2 / torch paths unchanged.

UPSTREAM REFERENCES (fixed after vcs import revealed actual names)
  - scout_piper_bringup/package.xml:
      piper_control -> piper_humble
      piper_moveit  -> piper_with_gripper_moveit
      added piper_description, piper_msgs, scout_description, scout_msgs,
      realsense2_description as exec_deps
  - scout_piper_bringup/launch/full_system.launch.py:
      piper_moveit/demo.launch.py -> piper_with_gripper_moveit/demo.launch.py
      scout_nav2/navigation.launch.py -> scout_nav2/nav2.launch.py
  - scout_piper_description/urdf/scout_piper.urdf.xacro:
      v0 = Scout-only. Upstream piper_description.xacro hardcodes
      base_link + world with no prefix arg; xacro:include collides with
      scout_v2.xacro. Documented P0.2.3 follow-up to fork the piper xacro
      with prefixed link names.

DOCKER DEV ENVIRONMENT (Ubuntu 20.04 host has no ros-humble apt packages)
  - docker/Dockerfile.dev:    osrf/ros:humble-desktop-full + MoveIt 2 +
                              ros2_control + nav2 + realsense2_camera +
                              moveit_py + python ML deps (numpy/scipy/
                              skimage/sklearn/open3d/ultralytics).
  - docker/compose.dev.yml:   GPU runtime, X11, host net, USB passthrough,
                              workspace bind-mount at /workspace.
  - docker/build_dev.sh:      one-shot builder.
  - docker/README.md:         daily-use docs.
  - scripts/install_docker_nvidia.sh:
                              installs Docker CE + nvidia-container-toolkit
                              on Ubuntu 20.04 (user supplies sudo).

WORKSPACE
  - vcstool + colcon installed via pip3 --user on the host (no sudo).
  - vcs import ran successfully: piper_ros@humble, scout_ros2@humble,
    scout_nav2@main, realsense-ros@ros2-development (~24 packages total
    discoverable by colcon).

PROGRESS.md updated for P0.1, P0.2.3 (blocked), P0.4.15-16 ports.

File: Codes/src/scout_piper_description/urdf/scout_piper.urdf.xacro (robot description, xacro)
@@ -3,46 +3,34 @@
   <!--
     Unified URDF for AgileX Piper 6-DoF arm mounted on Scout 2.0 UGV.
-    Composes three upstream URDFs:
-      - scout_description       : Scout 2.0 base
-      - piper_description       : Piper 6-DoF arm + gripper
-      - realsense2_description  : RealSense camera (eye-in-hand)
-    TF tree (high level):
-        map  ->  odom  ->  base_link (Scout)  ->  scout_top_plate
-              ->  piper_mount_link  ->  base_link (Piper)  -> ... -> link6
-              ->  realsense_link
-    The Scout's "base_link" is the kinematic root; the Piper's URDF also uses
-    "base_link" as its root, so we remap the Piper subtree's prefix via xacro
-    (piper_prefix) to avoid TF name collisions.
-    NOTE: This xacro DEPENDS on the upstream piper_description and
-    scout_description xacros being available after `vcs import`. If those
-    paths drift, update the xacro:include block below.
+    STATUS (2026-05-17):
+      v0 — Scout-only. The upstream agilexrobotics/piper_ros@humble ships a
+      piper_description.xacro that hardcodes its root as <link name="base_link"/>
+      AND defines a <link name="world"/> with a fixed joint to base_link. There
+      is no `prefix` argument on the upstream xacro, so xacro:include-ing it
+      alongside scout_v2.xacro produces a duplicate-link error.
+    TODO(P0.2.3): Fork piper_description.xacro into our own
+      scout_piper_description/urdf/_piper_arm.xacro with:
+        - all links prefixed (e.g., piper_base_link, piper_link1, …, piper_link6)
+        - the upstream world link + fixed_base_joint removed
+        - the upstream <link name="base_link"> renamed to piper_base_link
+      Then mount it on Scout via a fixed joint from base_link → piper_mount_link
+      → piper_base_link.
+    This v0 keeps view_robot.launch.py functional (you can verify the Scout
+    chassis + RealSense mount frame) while we sort out the arm integration.
   -->
   <xacro:arg name="use_sim"        default="false"/>
   <xacro:arg name="use_gazebo_ros" default="false"/>
-  <!-- ============================================================ -->
-  <!-- 1. Scout 2.0 base                                            -->
-  <!-- ============================================================ -->
-  <!-- Upstream Scout xacro provides links: base_link, base_footprint,
-       and four wheel links. We keep its default frame names. -->
+  <!-- Scout 2.0 base -->
   <xacro:include filename="$(find scout_description)/urdf/scout_v2.xacro"/>
-  <!-- ============================================================ -->
-  <!-- 2. Mount plate on Scout for the Piper arm                    -->
-  <!--    Adjust the xyz/rpy if the physical mount differs.         -->
-  <!-- ============================================================ -->
+  <!-- Piper mount plate (placeholder; tune dimensions to match the physical mount) -->
   <xacro:property name="piper_mount_xyz" value="0.15 0.0 0.18"/>
   <xacro:property name="piper_mount_rpy" value="0.0 0.0 0.0"/>
   <link name="piper_mount_link">
     <visual>
-      <geometry>
-        <box size="0.08 0.08 0.01"/>
-      </geometry>
-      <material name="aluminum">
-        <color rgba="0.7 0.7 0.7 1.0"/>
-      </material>
+      <geometry><box size="0.08 0.08 0.01"/></geometry>
+      <material name="aluminum"><color rgba="0.7 0.7 0.7 1.0"/></material>
     </visual>
     <collision>
-      <geometry>
-        <box size="0.08 0.08 0.01"/>
-      </geometry>
+      <geometry><box size="0.08 0.08 0.01"/></geometry>
     </collision>
     <inertial>
@@ -56,32 +44,10 @@
     <origin xyz="${piper_mount_xyz}" rpy="${piper_mount_rpy}"/>
   </joint>
-  <!-- ============================================================ -->
-  <!-- 3. Piper 6-DoF arm + gripper                                 -->
-  <!--    We re-prefix the Piper subtree to avoid base_link clash.  -->
-  <!--    Upstream piper_description supports a ${prefix} arg in    -->
-  <!--    most versions; if not, this xacro:include will need to be -->
-  <!--    swapped for a prefixed copy in this package's urdf/ dir.  -->
-  <!-- ============================================================ -->
-  <xacro:property name="piper_prefix" value="piper_"/>
-  <!-- Upstream path; verify after `vcs import` and update if needed. -->
-  <xacro:include filename="$(find piper_description)/urdf/piper_with_gripper.urdf.xacro"/>
-  <!-- The included xacro defines its own base_link as the arm's root.
-       We weld it onto the mount plate. If the upstream macro exposes a
-       prefix argument, prefer instantiating with prefix="${piper_prefix}"
-       and adjust this joint accordingly. -->
-  <joint name="piper_mount_to_piper_base" type="fixed">
-    <parent link="piper_mount_link"/>
-    <child  link="base_link"/>
-    <origin xyz="0 0 0.005" rpy="0 0 0"/>
-  </joint>
-  <!-- ============================================================ -->
-  <!-- 4. RealSense camera, eye-in-hand on Piper link6              -->
-  <!-- ============================================================ -->
-  <!-- These come from the hand-eye calibration; populate them in
-       config/hand_eye.yaml and override via xacro args at launch. -->
+  <!-- RealSense D435 (eye-in-hand placeholder until P0.2.3 is done). Mounted
+       on piper_mount_link for now so RViz shows a sensible camera frame. -->
   <xacro:arg name="cam_xyz" default="0.05 0.0 0.05"/>
   <xacro:arg name="cam_rpy" default="0.0 0.0 0.0"/>
   <xacro:include filename="$(find realsense2_description)/urdf/_d435.urdf.xacro"/>
-  <xacro:sensor_d435 name="camera" parent="link6" use_nominal_extrinsics="true">
+  <xacro:sensor_d435 name="camera" parent="piper_mount_link" use_nominal_extrinsics="true">
     <origin xyz="$(arg cam_xyz)" rpy="$(arg cam_rpy)"/>
   </xacro:sensor_d435>

Commit message: P0.2.3: fork piper xacro and integrate into unified URDF
Upstream piper_description.xacro hardcodes its arm root as <link name="base_link"/>
and adds a <link name="world"/> with a fixed joint to it. Both clash with
scout_v2.xacro which also defines base_link, so xacro:include-ing both into
one robot fails with duplicate-link errors.

scripts/fork_piper_arm.py:
  - Reads upstream piper_description.xacro
  - Strips XML header, robot opening/closing, the world link + fixed_base_joint
  - Adds ${prefix} to every link/joint/transmission/gazebo-reference name
  - Wraps everything in a <xacro:macro name="piper_arm"
    params="prefix parent *origin"> so the caller picks both the namespace
    and the parent link
  - Prepends a ${prefix}base_mount fixed joint inside the macro
  - Writes scout_piper_description/urdf/_piper_arm.xacro

scout_piper.urdf.xacro:
  - Instantiates the macro with prefix="piper_", parent="piper_mount_link"
  - Moves the RealSense D435 mount from piper_mount_link to piper_link6
    (proper eye-in-hand placement)

Verified: 10 links + 10 joints + 8 transmissions + 8 gazebo refs all carry
the piper_ prefix. The fork is idempotent — re-run the script whenever
upstream changes.

File: Codes/src/scout_piper_description/urdf/scout_piper.urdf.xacro (robot description, xacro)
@@ -2,28 +2,32 @@
 <robot name="scout_piper" xmlns:xacro="http://www.ros.org/wiki/xacro">
   <!--
-    Unified URDF for AgileX Piper 6-DoF arm mounted on Scout 2.0 UGV.
-    STATUS (2026-05-17):
-      v0 — Scout-only. The upstream agilexrobotics/piper_ros@humble ships a
-      piper_description.xacro that hardcodes its root as <link name="base_link"/>
-      AND defines a <link name="world"/> with a fixed joint to base_link. There
-      is no `prefix` argument on the upstream xacro, so xacro:include-ing it
-      alongside scout_v2.xacro produces a duplicate-link error.
-    TODO(P0.2.3): Fork piper_description.xacro into our own
-      scout_piper_description/urdf/_piper_arm.xacro with:
-        - all links prefixed (e.g., piper_base_link, piper_link1, …, piper_link6)
-        - the upstream world link + fixed_base_joint removed
-        - the upstream <link name="base_link"> renamed to piper_base_link
-      Then mount it on Scout via a fixed joint from base_link → piper_mount_link
-      → piper_base_link.
-    This v0 keeps view_robot.launch.py functional (you can verify the Scout
-    chassis + RealSense mount frame) while we sort out the arm integration.
+    Unified URDF for AgileX Piper 6-DoF arm mounted on Scout 2.0 UGV with an
+    eye-in-hand RealSense D435.
+    Composes three subtrees:
+      1. Scout 2.0 base       — upstream scout_description (root link: base_link)
+      2. Piper arm + gripper  — forked piper_description, prefixed `piper_` and
+                                wrapped in a macro (see _piper_arm.xacro)
+      3. RealSense D435       — upstream realsense2_description, mounted on
+                                piper_link6 (the EE flange)
+    TF tree:
+      odom -> base_link (Scout) -> piper_mount_link -> piper_base_link
+              -> piper_link1 -> ... -> piper_link6 -> camera_link
+                                                  \-> piper_gripper_base
+                                                        \-> piper_link7
+                                                        \-> piper_link8
   -->
   <xacro:arg name="use_sim"        default="false"/>
   <xacro:arg name="use_gazebo_ros" default="false"/>
-  <!-- Scout 2.0 base -->
+  <!-- Eye-in-hand camera placement on the EE flange. Override at launch
+       once hand-eye calibration is done. -->
+  <xacro:arg name="cam_xyz" default="0.05 0.0 0.05"/>
+  <xacro:arg name="cam_rpy" default="0.0 0.0 0.0"/>
+  <!-- =========================================================== -->
+  <!-- 1. Scout 2.0 base                                            -->
+  <!-- =========================================================== -->
   <xacro:include filename="$(find scout_description)/urdf/scout_v2.xacro"/>
-  <!-- Piper mount plate (placeholder; tune dimensions to match the physical mount) -->
-  <xacro:property name="piper_mount_xyz" value="0.15 0.0 0.18"/>
-  <xacro:property name="piper_mount_rpy" value="0.0 0.0 0.0"/>
+  <!-- =========================================================== -->
+  <!-- 2. Piper mount plate (placeholder; tune to physical mount)   -->
+  <!-- =========================================================== -->
   <link name="piper_mount_link">
     <visual>
@@ -42,12 +46,18 @@
     <parent link="base_link"/>
     <child  link="piper_mount_link"/>
-    <origin xyz="${piper_mount_xyz}" rpy="${piper_mount_rpy}"/>
+    <origin xyz="0.15 0.0 0.18" rpy="0 0 0"/>
   </joint>
-  <!-- RealSense D435 (eye-in-hand placeholder until P0.2.3 is done). Mounted
-       on piper_mount_link for now so RViz shows a sensible camera frame. -->
-  <xacro:arg name="cam_xyz" default="0.05 0.0 0.05"/>
-  <xacro:arg name="cam_rpy" default="0.0 0.0 0.0"/>
+  <!-- =========================================================== -->
+  <!-- 3. Piper 6-DoF arm + gripper (forked macro)                  -->
+  <!-- =========================================================== -->
+  <xacro:include filename="$(find scout_piper_description)/urdf/_piper_arm.xacro"/>
+  <xacro:piper_arm prefix="piper_" parent="piper_mount_link">
+    <origin xyz="0 0 0.005" rpy="0 0 0"/>
+  </xacro:piper_arm>
+  <!-- =========================================================== -->
+  <!-- 4. RealSense D435 (eye-in-hand on the EE flange)             -->
+  <!-- =========================================================== -->
   <xacro:include filename="$(find realsense2_description)/urdf/_d435.urdf.xacro"/>
-  <xacro:sensor_d435 name="camera" parent="piper_mount_link" use_nominal_extrinsics="true">
+  <xacro:sensor_d435 name="camera" parent="piper_link6" use_nominal_extrinsics="true">
     <origin xyz="$(arg cam_xyz)" rpy="$(arg cam_rpy)"/>
   </xacro:sensor_d435>
